File: dac.sch (KiCad schematic (older format))
At the start: 19 parts, among them J1 RCA-Connector, SW1 SW_DIP_x01, U1 pcm5102a

Commit message: termine esquematico
Parts:
- added J2: Conn_01x03_Male, symbol Connector:Conn_01x03_Male
- U1: symbol pcm5102a-rescue:pcm5102a -> dac-rescue:pcm5102a-pcm5102a-rescue
Connections:
- net labels added: +3.3VA, Earth, GNDA
- wire segments 60 -> 76
Other:
- note added: "I2S_BCK"
- note added: "I2S_LRCK"
- note added: "I2S_SDOUT"
- note added: "Left Channel Line Output"
- note added: "Right Channel Line Output"
- moved on the sheet: C6, C8, J1
