File: dac.sch (KiCad schematic (older format))
At the start: 20 parts, among them J1 RCA-Connector, J2 Conn_01x03_Male, SW1 SW_DIP_x01, U1 pcm5102a

Commit message: start PCB
Parts:
- removed J1: RCA-Connector, symbol Connector:Conn_Coaxial_x2
- added J1, J3: RCA, tp-fvbattocchia:CUI_RCJ-013, symbol RCJ-013:RCJ-013
Connections:
- wire segments 76 -> 77
Other:
- moved on the sheet: C12, C13
Changed lines of the file:
@@
 L Device:C C12
 U 1 1 604E712E
-P 6650 3400
-F 0 "C12" H 6765 3446 50  0000 L CNN
-F 1 "2.2nF" H 6765 3355 50  0000 L CNN
-F 2 "Capacitor_THT:C_Disc_D3.0mm_W1.6mm_P2.50mm" H 6688 3250 50  0001 C CNN
-F 3 "~" H 6650 3400 50  0001 C CNN
-	1    6650 3400
+P 7150 3300
+F 0 "C12" H 7265 3346 50  0000 L CNN
+F 1 "2.2nF" H 7265 3255 50  0000 L CNN
+F 2 "Capacitor_THT:C_Disc_D3.0mm_W1.6mm_P2.50mm" H 7188 3150 50  0001 C CNN
+F 3 "~" H 7150 3300 50  0001 C CNN
+	1    7150 3300
 	1    0    0    -1
 $EndComp
@@
 	5450 3150 6300 3150
 Wire Wire Line
-	6600 3150 6650 3150
-Wire Wire Line
-	6650 3250 6650 3150
-Connection ~ 6650 3150
-Wire Wire Line
 	6050 2550 6050 2600
 Wire Wire Line
@@
 Wire Wire Line
 	5450 2850 5550 2850
-Wire Wire Line
-	7100 3050 7100 2950
-Text Notes 7650 2950 0    50   ~ 0
+Text Notes 8150 2900 0    50   ~ 0
 Right Channel Line Output
-Text Notes 7650 3300 0    50   ~ 0
+Text Notes 8150 3450 0    50   ~ 0
 Left Channel Line Output
-$Comp
-L power:GNDA #PWR012
-U 1 1 6056AD9C
-P 7500 3350
-F 0 "#PWR012" H 7500 3100 50  0001 C CNN
-F 1 "GNDA" H 7505 3177 50  0000 C CNN
-F 2 "" H 7500 3350 50  0001 C CNN
-F 3 "" H 7500 3350 50  0001 C CNN
-	1    7500 3350
-	1    0    0    -1
-$EndComp
 $Comp
 L power:GNDA #PWR07
 U 1 1 6056EE96
-P 6650 3550
-F 0 "#PWR07" H 6650 3300 50  0001 C CNN
-F 1 "GNDA" H 6655 3377 50  0000 C CNN
-F 2 "" H 6650 3550 50  0001 C CNN
-F 3 "" H 6650 3550 50  0001 C CNN
-	1    6650 3550
-	1    0    0    -1
-$EndComp
-$Comp
-L Connector:Conn_Coaxial_x2 J1
-U 1 1 604DAEE2
-P 7500 3050
-F 0 "J1" H 7600 3025 50  0000 L CNN
-F 1 "RCA-Connector" H 7600 2934 50  0000 L CNN
-F 2 "" H 7500 2950 50  0001 C CNN
-F 3 " ~" H 7500 2950 50  0001 C CNN
-	1    7500 3050
+P 7500 3450
+F 0 "#PWR07" H 7500 3200 50  0001 C CNN
+F 1 "GNDA" H 7505 3277 50  0000 C CNN
+F 2 "" H 7500 3450 50  0001 C CNN
+F 3 "" H 7500 3450 50  0001 C CNN
+	1    7500 3450
 	1    0    0    -1
 $EndComp
@@
 L Device:C C13
 U 1 1 604E73B9
-P 7100 3400
-F 0 "C13" H 7215 3446 50  0000 L CNN
-F 1 "2.2nF" H 7215 3355 50  0000 L CNN
-F 2 "Capacitor_THT:C_Disc_D3.0mm_W1.6mm_P2.50mm" H 7138 3250 50  0001 C CNN
-F 3 "~" H 7100 3400 50  0001 C CNN
-	1    7100 3400
-	1    0    0    -1
-$EndComp
-Wire Wire Line
-	6600 3050 7100 3050
-Wire Wire Line
-	7100 2950 7300 2950
+P 7150 2900
+F 0 "C13" H 7265 2946 50  0000 L CNN
+F 1 "2.2nF" H 7265 2855 50  0000 L CNN
+F 2 "Capacitor_THT:C_Disc_D3.0mm_W1.6mm_P2.50mm" H 7188 2750 50  0001 C CNN
+F 3 "~" H 7150 2900 50  0001 C CNN
+	1    7150 2900
+	-1   0    0    1
+$EndComp
 $Comp
 L power:GNDA #PWR011
 U 1 1 6059B373
-P 7100 3550
-F 0 "#PWR011" H 7100 3300 50  0001 C CNN
-F 1 "GNDA" H 7105 3377 50  0000 C CNN
-F 2 "" H 7100 3550 50  0001 C CNN
-F 3 "" H 7100 3550 50  0001 C CNN
-	1    7100 3550
-	1    0    0    -1
-$EndComp
-Wire Wire Line
-	6650 3150 7300 3150
-Wire Wire Line
-	7100 3250 7100 3050
-Connection ~ 7100 3050
+P 7500 2750
+F 0 "#PWR011" H 7500 2500 50  0001 C CNN
+F 1 "GNDA" H 7505 2577 50  0000 C CNN
+F 2 "" H 7500 2750 50  0001 C CNN
+F 3 "" H 7500 2750 50  0001 C CNN
+	1    7500 2750
+	-1   0    0    1
+$EndComp
 $Comp
 L power:GNDA #PWR09
@@
 	6500 3750 6500 3850
 Connection ~ 6500 3850
+$Comp
+L RCJ-013:RCJ-013 J1
+U 1 1 6065BCFC
+P 7800 2950
+F 0 "J1" H 7642 2916 50  0000 R CNN
+F 1 "RCA" H 7642 3007 50  0000 R CNN
+F 2 "tp-fvbattocchia:CUI_RCJ-013" H 7800 2950 50  0001 L BNN
+F 3 "" H 7800 2950 50  0001 L BNN
+F 4 "Manufacturer recommendations" H 7800 2950 50  0001 L BNN "STANDARD"
+F 5 "CUI Inc" H 7800 2950 50  0001 L BNN "MANUFACTURER"
+F 6 "B" H 7800 2950 50  0001 L BNN "PART_REV"
+	1    7800 2950
+	-1   0    0    1
+$EndComp
+$Comp
+L RCJ-013:RCJ-013 J3
+U 1 1 6065E5C6
+P 7800 3250
+F 0 "J3" H 7642 3216 50  0000 R CNN
+F 1 "RCA" H 7642 3307 50  0000 R CNN
+F 2 "tp-fvbattocchia:CUI_RCJ-013" H 7800 3250 50  0001 L BNN
+F 3 "" H 7800 3250 50  0001 L BNN
+F 4 "Manufacturer recommendations" H 7800 3250 50  0001 L BNN "STANDARD"
+F 5 "CUI Inc" H 7800 3250 50  0001 L BNN "MANUFACTURER"
+F 6 "B" H 7800 3250 50  0001 L BNN "PART_REV"
+	1    7800 3250
+	-1   0    0    1
+$EndComp
+Wire Wire Line
+	6600 3050 7150 3050
+Wire Wire Line
+	7500 2750 7500 2850
+Connection ~ 7500 2750
+Connection ~ 7150 3150
+Wire Wire Line
+	7150 3150 7500 3150
+Wire Wire Line
+	6600 3150 7150 3150
+Wire Wire Line
+	7500 3350 7500 3450
+Wire Wire Line
+	7500 3450 7150 3450
+Connection ~ 7150 3050
+Wire Wire Line
+	7150 3050 7500 3050
+Wire Wire Line
+	7150 2750 7500 2750
+Connection ~ 7500 3450
 $EndSCHEMATC

Commit message: se corrije esquematico y pcb conector RCA, se agrega modelo 3d
Parts:
- removed J1, J3: RCA, tp-fvbattocchia:CUI_RCJ-013, symbol RCJ-013:RCJ-013
- added J1: RCJ-2121, RCJ-2121:RCJ-2121, symbol RCJ-2121:RCJ-2121
Connections:
- wire segments 77 -> 79

Commit message: correcciones
Connections:
- wire segments 79 -> 81
Changed lines of the file:
@@
 encoding utf-8
 Sheet 1 1
-Title "Modulo Pcm5102a 5102 Decodificador Stereo Audio Digital"
+Title "Modulo Pcm5102a Decodificador Stereo Audio Digital"
 Date "2021-03-13"
-Rev ""
+Rev "Pablo Aguirre"
 Comp "Florencia Battocchia - Diseño de PCB -CESE"
 Comment1 ""
@@
 U 1 1 604E6F3C
 P 3800 3600
-F 0 "C3" H 3915 3646 50  0000 L CNN
-F 1 "0.1uF" H 3915 3555 50  0000 L CNN
+F 0 "C3" H 3550 3650 50  0000 L CNN
+F 1 "0.1uF" H 3500 3550 50  0000 L CNN
 F 2 "Capacitor_THT:C_Disc_D3.8mm_W2.6mm_P2.50mm" H 3838 3450 50  0001 C CNN
 F 3 "~" H 3800 3600 50  0001 C CNN
@@
 U 1 1 604E99FE
 P 3350 3600
-F 0 "C1" H 3441 3646 50  0000 L CNN
-F 1 "10uF" H 3441 3555 50  0000 L CNN
+F 0 "C1" H 3150 3650 50  0000 L CNN
+F 1 "10uF" H 3100 3550 50  0000 L CNN
 F 2 "Capacitor_THT:C_Radial_D4.0mm_H5.0mm_P1.50mm" H 3350 3600 50  0001 C CNN
 F 3 "~" H 3350 3600 50  0001 C CNN
@@
 U 1 1 604EA5B5
 P 6500 3950
-F 0 "C11" H 6591 3996 50  0000 L CNN
-F 1 "10uF" H 6591 3905 50  0000 L CNN
+F 0 "C11" H 6250 3900 50  0000 L CNN
+F 1 "10uF" H 6250 4000 50  0000 L CNN
 F 2 "Capacitor_THT:C_Radial_D4.0mm_H5.0mm_P1.50mm" H 6500 3950 50  0001 C CNN
 F 3 "~" H 6500 3950 50  0001 C CNN
 	1    6500 3950
-	1    0    0    -1
+	-1   0    0    1
 $EndComp
 Wire Wire Line
@@
 Wire Wire Line
 	3800 3750 3800 3800
-Wire Wire Line
-	3800 3800 3350 3800
 Connection ~ 3800 3800
 Connection ~ 3350 3800
 Wire Wire Line
 	3350 3800 3350 3700
-Wire Wire Line
-	3800 3450 3350 3450
 Wire Wire Line
 	3350 3450 3350 3500
@@
 P 6100 3950
 F 0 "C10" H 6215 3996 50  0000 L CNN
-F 1 "0.1uF" H 6215 3905 50  0000 L CNN
+F 1 "0.1uF" H 6200 3900 50  0000 L CNN
 F 2 "Capacitor_THT:C_Disc_D3.8mm_W2.6mm_P2.50mm" H 6138 3800 50  0001 C CNN
 F 3 "~" H 6100 3950 50  0001 C CNN
@@
 	5650 2950 5650 2850
 Wire Wire Line
-	5650 2850 6050 2850
-Wire Wire Line
 	6050 2850 6050 2800
 Connection ~ 5650 2850
@@
 	4400 3550 4150 3550
 Wire Wire Line
-	3800 3450 4400 3450
+	3800 3450 4100 3450
 Wire Wire Line
 	3200 3350 4400 3350
@@
 Wire Wire Line
 	6500 3750 6500 3850
-Connection ~ 6500 3850
 Wire Wire Line
 	6600 3150 7150 3150
@@
 Connection ~ 7350 2750
 Connection ~ 7350 3450
+Connection ~ 6500 3850
+$Comp
+L power:PWR_FLAG #FLG0101
+U 1 1 60790EFD
+P 5650 2950
+F 0 "#FLG0101" H 5650 3025 50  0001 C CNN
+F 1 "PWR_FLAG" V 5650 3078 50  0000 L CNN
+F 2 "" H 5650 2950 50  0001 C CNN
+F 3 "~" H 5650 2950 50  0001 C CNN
+	1    5650 2950
+	0    1    1    0
+$EndComp
+$Comp
+L power:PWR_FLAG #FLG0102
+U 1 1 60797BB9
+P 4100 3450
+F 0 "#FLG0102" H 4100 3525 50  0001 C CNN
+F 1 "PWR_FLAG" H 4100 3400 50  0000 C CNN
+F 2 "" H 4100 3450 50  0001 C CNN
+F 3 "~" H 4100 3450 50  0001 C CNN
+	1    4100 3450
+	-1   0    0    1
+$EndComp
+Wire Wire Line
+	3350 3800 3800 3800
+Wire Wire Line
+	3350 3450 3800 3450
+Connection ~ 4100 3450
+Wire Wire Line
+	4100 3450 4400 3450
+Connection ~ 5650 2950
+Wire Wire Line
+	5650 2850 6050 2850
+$Comp
+L power:PWR_FLAG #FLG0103
+U 1 1 607F3801
+P 7150 2550
+F 0 "#FLG0103" H 7150 2625 50  0001 C CNN
+F 1 "PWR_FLAG" H 7150 2723 50  0000 C CNN
+F 2 "" H 7150 2550 50  0001 C CNN
+F 3 "~" H 7150 2550 50  0001 C CNN
+	1    7150 2550
+	1    0    0    -1
+$EndComp
+Wire Wire Line
+	7150 2550 7150 2750
+Connection ~ 7150 2750
+$Comp
+L power:PWR_FLAG #FLG0104
+U 1 1 607F9605
+P 3100 3800
+F 0 "#FLG0104" H 3100 3875 50  0001 C CNN
+F 1 "PWR_FLAG" V 3100 3927 50  0000 L CNN
+F 2 "" H 3100 3800 50  0001 C CNN
+F 3 "~" H 3100 3800 50  0001 C CNN
+	1    3100 3800
+	0    -1   -1   0
+$EndComp
+Connection ~ 3100 3800
 $EndSCHEMATC

Commit message: se avanza en el pcb
Parts:
- added FID1: Fiducial, Fiducial:Fiducial_0.5mm_Mask1.5mm, symbol Mechanical:Fiducial
- C1, C11, C2, C8: footprint Capacitor_THT:C_Radial_D4.0mm_H5.0mm_P1.50mm -> Capacitor_THT:CP_Radial_D4.0mm_P1.50mm
Changed lines of the file:
@@
 F 0 "C1" H 3150 3650 50  0000 L CNN
 F 1 "10uF" H 3100 3550 50  0000 L CNN
-F 2 "Capacitor_THT:C_Radial_D4.0mm_H5.0mm_P1.50mm" H 3350 3600 50  0001 C CNN
+F 2 "Capacitor_THT:CP_Radial_D4.0mm_P1.50mm" H 3350 3600 50  0001 C CNN
 F 3 "~" H 3350 3600 50  0001 C CNN
 	1    3350 3600
@@
 F 0 "C8" H 5959 2654 50  0000 R CNN
 F 1 "10uF" H 5959 2745 50  0000 R CNN
-F 2 "Capacitor_THT:C_Radial_D4.0mm_H5.0mm_P1.50mm" H 6050 2700 50  0001 C CNN
+F 2 "Capacitor_THT:CP_Radial_D4.0mm_P1.50mm" H 6050 2700 50  0001 C CNN
 F 3 "~" H 6050 2700 50  0001 C CNN
 	1    6050 2700
@@
 F 0 "C2" H 3259 3904 50  0000 R CNN
 F 1 "10uF" H 3259 3995 50  0000 R CNN
-F 2 "Capacitor_THT:C_Radial_D4.0mm_H5.0mm_P1.50mm" H 3350 3950 50  0001 C CNN
+F 2 "Capacitor_THT:CP_Radial_D4.0mm_P1.50mm" H 3350 3950 50  0001 C CNN
 F 3 "~" H 3350 3950 50  0001 C CNN
 	1    3350 3950
@@
 F 0 "C11" H 6250 3900 50  0000 L CNN
 F 1 "10uF" H 6250 4000 50  0000 L CNN
-F 2 "Capacitor_THT:C_Radial_D4.0mm_H5.0mm_P1.50mm" H 6500 3950 50  0001 C CNN
+F 2 "Capacitor_THT:CP_Radial_D4.0mm_P1.50mm" H 6500 3950 50  0001 C CNN
 F 3 "~" H 6500 3950 50  0001 C CNN
 	1    6500 3950
@@
 $EndComp
 Connection ~ 3100 3800
+$Comp
+L Mechanical:Fiducial FID1
+U 1 1 6077A9FA
+P 5300 3850
+F 0 "FID1" H 5150 3750 50  0000 L CNN
+F 1 "Fiducial" H 5150 3700 50  0000 L CNN
+F 2 "Fiducial:Fiducial_0.5mm_Mask1.5mm" H 5300 3850 50  0001 C CNN
+F 3 "~" H 5300 3850 50  0001 C CNN
+	1    5300 3850
+	1    0    0    -1
+$EndComp
 $EndSCHEMATC

Commit message: correcciones en el esquematico indicadas  por el profesor
Parts:
- J1: Número de cátalogo (none) -> CP-1430-ND
- SW1: Código de catálogo en Digikey. (none) -> EG5071-ND
- U1: Código de catálogo en Digikey. (none) -> 296-36705-2-ND
Connections:
- net labels added: FLT, GND, OUTL, OUTR
- net labels removed: Earth
- wire segments 81 -> 77
Other:
- note added: "Conexiones del CI"
- note added: "output circuit"
- moved on the sheet: C1, C10, C11, C12, C13, C2, C3, C4, C5, C6, C7, C8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

Commit message: pcb terminado
Parts:
- added J3: Conn_01x02_Male, Connector_PinHeader_2.54mm:PinHeader_1x02_P2.54mm_Vertical, symbol Connector:Conn_01x02_Male
Connections:
- net +3.3VA: now also J3.1 (Pin_1)
- net GNDA: now also J3.2 (Pin_2)
Changed lines of the file:
@@
 Wire Wire Line
 	6550 4150 6550 4350
-Text Notes 3600 3700 0    50   ~ 0
+Text Notes 4800 3650 0    50   ~ 0
 Conexiones del CI
 Wire Wire Line
@@
 Wire Wire Line
 	5750 5400 5750 5300
+Wire Wire Line
+	4850 2150 5200 2150
+Wire Notes Line
+	3500 3050 5900 3050
+Wire Notes Line
+	3500 1600 5900 1600
+$Comp
+L power:+3.3VA #PWR0104
+U 1 1 60A48341
+P 4450 3900
+F 0 "#PWR0104" H 4450 3750 50  0001 C CNN
+F 1 "+3.3VA" V 4450 4150 50  0000 C CNN
+F 2 "" H 4450 3900 50  0001 C CNN
+F 3 "" H 4450 3900 50  0001 C CNN
+	1    4450 3900
+	0    1    1    0
+$EndComp
+$Comp
+L power:PWR_FLAG #FLG0101
+U 1 1 60790EFD
+P 4350 3850
+F 0 "#FLG0101" H 4350 3925 50  0001 C CNN
+F 1 "PWR_FLAG" H 4350 3978 50  0000 L CNN
+F 2 "" H 4350 3850 50  0001 C CNN
+F 3 "~" H 4350 3850 50  0001 C CNN
+	1    4350 3850
+	1    0    0    -1
+$EndComp
+$Comp
+L power:PWR_FLAG #FLG0102
+U 1 1 60A4D20D
+P 4350 4050
+F 0 "#FLG0102" H 4350 4125 50  0001 C CNN
+F 1 "PWR_FLAG" H 3950 4200 50  0000 L CNN
+F 2 "" H 4350 4050 50  0001 C CNN
+F 3 "~" H 4350 4050 50  0001 C CNN
+	1    4350 4050
+	-1   0    0    1
+$EndComp
+$Comp
+L power:GNDA #PWR0103
+U 1 1 60A3D0B2
+P 4450 4000
+F 0 "#PWR0103" H 4450 3750 50  0001 C CNN
+F 1 "GNDA" V 4450 3800 50  0000 C CNN
+F 2 "" H 4450 4000 50  0001 C CNN
+F 3 "" H 4450 4000 50  0001 C CNN
+	1    4450 4000
+	0    -1   -1   0
+$EndComp
+$Comp
+L Connector:Conn_01x02_Male J3
+U 1 1 607E48C9
+P 4050 3900
+F 0 "J3" H 4158 4081 50  0000 C CNN
+F 1 "Conn_01x02_Male" H 3900 4000 50  0000 C CNN
+F 2 "Connector_PinHeader_2.54mm:PinHeader_1x02_P2.54mm_Vertical" H 4050 3900 50  0001 C CNN
+F 3 "~" H 4050 3900 50  0001 C CNN
+	1    4050 3900
+	1    0    0    -1
+$EndComp
+Wire Wire Line
+	4250 3900 4350 3900
+Wire Wire Line
+	4250 4000 4350 4000
+Wire Wire Line
+	4350 3850 4350 3900
+Connection ~ 4350 3900
+Wire Wire Line
+	4350 3900 4450 3900
+Wire Wire Line
+	4350 4050 4350 4000
+Connection ~ 4350 4000
+Wire Wire Line
+	4350 4000 4450 4000
 $Comp
 L power:PWR_FLAG #FLG0104
@@
 Wire Wire Line
 	5650 5400 5750 5400
-Wire Wire Line
-	4850 2150 5200 2150
-Wire Notes Line
-	3500 3050 5900 3050
-Wire Notes Line
-	3500 1600 5900 1600
-Wire Wire Line
-	6900 3750 6900 3850
-$Comp
-L power:+3.3VA #PWR0104
-U 1 1 60A48341
-P 6900 3850
-F 0 "#PWR0104" H 6900 3700 50  0001 C CNN
-F 1 "+3.3VA" H 6915 4023 50  0000 C CNN
-F 2 "" H 6900 3850 50  0001 C CNN
-F 3 "" H 6900 3850 50  0001 C CNN
-	1    6900 3850
-	-1   0    0    1
-$EndComp
-$Comp
-L power:PWR_FLAG #FLG0101
-U 1 1 60790EFD
-P 6900 3750
-F 0 "#FLG0101" H 6900 3825 50  0001 C CNN
-F 1 "PWR_FLAG" H 6900 3878 50  0000 L CNN
-F 2 "" H 6900 3750 50  0001 C CNN
-F 3 "~" H 6900 3750 50  0001 C CNN
-	1    6900 3750
-	1    0    0    -1
-$EndComp
-Wire Wire Line
-	7500 3750 7500 3850
-$Comp
-L power:PWR_FLAG #FLG0102
-U 1 1 60A4D20D
-P 7500 3750
-F 0 "#FLG0102" H 7500 3825 50  0001 C CNN
-F 1 "PWR_FLAG" H 7500 3878 50  0000 L CNN
-F 2 "" H 7500 3750 50  0001 C CNN
-F 3 "~" H 7500 3750 50  0001 C CNN
-	1    7500 3750
-	1    0    0    -1
-$EndComp
-$Comp
-L power:GNDA #PWR0103
-U 1 1 60A3D0B2
-P 7500 3850
-F 0 "#PWR0103" H 7500 3600 50  0001 C CNN
-F 1 "GNDA" H 7505 3677 50  0000 C CNN
-F 2 "" H 7500 3850 50  0001 C CNN
-F 3 "" H 7500 3850 50  0001 C CNN
-	1    7500 3850
-	1    0    0    -1
-$EndComp
 $EndSCHEMATC

Commit message: correcciones pcb
Parts:
- added H1: MountingHole, MountingHole:MountingHole_2.5mm, symbol Mechanical:MountingHole
Changed lines of the file:
@@
 Wire Wire Line
 	5650 5400 5750 5400
+$Comp
+L Mechanical:MountingHole H1
+U 1 1 608A30DB
+P 7150 3700
+F 0 "H1" H 7250 3746 50  0000 L CNN
+F 1 "MountingHole" H 7250 3655 50  0000 L CNN
+F 2 "MountingHole:MountingHole_2.5mm" H 7150 3700 50  0001 C CNN
+F 3 "~" H 7150 3700 50  0001 C CNN
+	1    7150 3700
+	1    0    0    -1
+$EndComp
 $EndSCHEMATC
