File: _autosave-dac.sch (KiCad schematic (older format))
At the start: 20 parts, among them J1 RCA-Connector, J2 Conn_01x03_Male, SW1 SW_DIP_x01, U1 pcm5102a

Commit message: start PCB
Parts:
- removed J1: RCA-Connector, symbol Connector:Conn_Coaxial_x2
- added J1, J3: RCA, CUI_RCJ-013, symbol RCJ-013:RCJ-013
Connections:
- wire segments 76 -> 77
Other:
- moved on the sheet: C12, C13
Changed lines of the file:
@@
 L Device:C C12
 U 1 1 604E712E
-P 6650 3400
-F 0 "C12" H 6765 3446 50  0000 L CNN
-F 1 "2.2nF" H 6765 3355 50  0000 L CNN
-F 2 "Capacitor_THT:C_Disc_D3.0mm_W1.6mm_P2.50mm" H 6688 3250 50  0001 C CNN
-F 3 "~" H 6650 3400 50  0001 C CNN
-	1    6650 3400
+P 7150 3300
+F 0 "C12" H 7265 3346 50  0000 L CNN
+F 1 "2.2nF" H 7265 3255 50  0000 L CNN
+F 2 "Capacitor_THT:C_Disc_D3.0mm_W1.6mm_P2.50mm" H 7188 3150 50  0001 C CNN
+F 3 "~" H 7150 3300 50  0001 C CNN
+	1    7150 3300
 	1    0    0    -1
 $EndComp
@@
 	5450 3150 6300 3150
 Wire Wire Line
-	6600 3150 6650 3150
-Wire Wire Line
-	6650 3250 6650 3150
-Connection ~ 6650 3150
-Wire Wire Line
 	6050 2550 6050 2600
 Wire Wire Line
@@
 Wire Wire Line
 	5450 2850 5550 2850
-Wire Wire Line
-	7100 3050 7100 2950
-Text Notes 7650 2950 0    50   ~ 0
+Text Notes 8150 2900 0    50   ~ 0
 Right Channel Line Output
-Text Notes 7650 3300 0    50   ~ 0
+Text Notes 8150 3450 0    50   ~ 0
 Left Channel Line Output
-$Comp
-L power:GNDA #PWR012
-U 1 1 6056AD9C
-P 7500 3350
-F 0 "#PWR012" H 7500 3100 50  0001 C CNN
-F 1 "GNDA" H 7505 3177 50  0000 C CNN
-F 2 "" H 7500 3350 50  0001 C CNN
-F 3 "" H 7500 3350 50  0001 C CNN
-	1    7500 3350
-	1    0    0    -1
-$EndComp
 $Comp
 L power:GNDA #PWR07
 U 1 1 6056EE96
-P 6650 3550
-F 0 "#PWR07" H 6650 3300 50  0001 C CNN
-F 1 "GNDA" H 6655 3377 50  0000 C CNN
-F 2 "" H 6650 3550 50  0001 C CNN
-F 3 "" H 6650 3550 50  0001 C CNN
-	1    6650 3550
-	1    0    0    -1
-$EndComp
-$Comp
-L Connector:Conn_Coaxial_x2 J1
-U 1 1 604DAEE2
-P 7500 3050
-F 0 "J1" H 7600 3025 50  0000 L CNN
-F 1 "RCA-Connector" H 7600 2934 50  0000 L CNN
-F 2 "" H 7500 2950 50  0001 C CNN
-F 3 " ~" H 7500 2950 50  0001 C CNN
-	1    7500 3050
+P 7500 3450
+F 0 "#PWR07" H 7500 3200 50  0001 C CNN
+F 1 "GNDA" H 7505 3277 50  0000 C CNN
+F 2 "" H 7500 3450 50  0001 C CNN
+F 3 "" H 7500 3450 50  0001 C CNN
+	1    7500 3450
 	1    0    0    -1
 $EndComp
@@
 L Device:C C13
 U 1 1 604E73B9
-P 7100 3400
-F 0 "C13" H 7215 3446 50  0000 L CNN
-F 1 "2.2nF" H 7215 3355 50  0000 L CNN
-F 2 "Capacitor_THT:C_Disc_D3.0mm_W1.6mm_P2.50mm" H 7138 3250 50  0001 C CNN
-F 3 "~" H 7100 3400 50  0001 C CNN
-	1    7100 3400
-	1    0    0    -1
-$EndComp
-Wire Wire Line
-	6600 3050 7100 3050
-Wire Wire Line
-	7100 2950 7300 2950
+P 7150 2900
+F 0 "C13" H 7265 2946 50  0000 L CNN
+F 1 "2.2nF" H 7265 2855 50  0000 L CNN
+F 2 "Capacitor_THT:C_Disc_D3.0mm_W1.6mm_P2.50mm" H 7188 2750 50  0001 C CNN
+F 3 "~" H 7150 2900 50  0001 C CNN
+	1    7150 2900
+	-1   0    0    1
+$EndComp
 $Comp
 L power:GNDA #PWR011
 U 1 1 6059B373
-P 7100 3550
-F 0 "#PWR011" H 7100 3300 50  0001 C CNN
-F 1 "GNDA" H 7105 3377 50  0000 C CNN
-F 2 "" H 7100 3550 50  0001 C CNN
-F 3 "" H 7100 3550 50  0001 C CNN
-	1    7100 3550
-	1    0    0    -1
-$EndComp
-Wire Wire Line
-	6650 3150 7300 3150
-Wire Wire Line
-	7100 3250 7100 3050
-Connection ~ 7100 3050
+P 7500 2750
+F 0 "#PWR011" H 7500 2500 50  0001 C CNN
+F 1 "GNDA" H 7505 2577 50  0000 C CNN
+F 2 "" H 7500 2750 50  0001 C CNN
+F 3 "" H 7500 2750 50  0001 C CNN
+	1    7500 2750
+	-1   0    0    1
+$EndComp
 $Comp
 L power:GNDA #PWR09
@@
 	6500 3750 6500 3850
 Connection ~ 6500 3850
+$Comp
+L RCJ-013:RCJ-013 J1
+U 1 1 6065BCFC
+P 7800 2950
+F 0 "J1" H 7642 2916 50  0000 R CNN
+F 1 "RCA" H 7642 3007 50  0000 R CNN
+F 2 "CUI_RCJ-013" H 7800 2950 50  0001 L BNN
+F 3 "" H 7800 2950 50  0001 L BNN
+F 4 "Manufacturer recommendations" H 7800 2950 50  0001 L BNN "STANDARD"
+F 5 "CUI Inc" H 7800 2950 50  0001 L BNN "MANUFACTURER"
+F 6 "B" H 7800 2950 50  0001 L BNN "PART_REV"
+	1    7800 2950
+	-1   0    0    1
+$EndComp
+$Comp
+L RCJ-013:RCJ-013 J3
+U 1 1 6065E5C6
+P 7800 3250
+F 0 "J3" H 7642 3216 50  0000 R CNN
+F 1 "RCA" H 7642 3307 50  0000 R CNN
+F 2 "CUI_RCJ-013" H 7800 3250 50  0001 L BNN
+F 3 "" H 7800 3250 50  0001 L BNN
+F 4 "Manufacturer recommendations" H 7800 3250 50  0001 L BNN "STANDARD"
+F 5 "CUI Inc" H 7800 3250 50  0001 L BNN "MANUFACTURER"
+F 6 "B" H 7800 3250 50  0001 L BNN "PART_REV"
+	1    7800 3250
+	-1   0    0    1
+$EndComp
+Wire Wire Line
+	6600 3050 7150 3050
+Wire Wire Line
+	7500 2750 7500 2850
+Connection ~ 7500 2750
+Connection ~ 7150 3150
+Wire Wire Line
+	7150 3150 7500 3150
+Wire Wire Line
+	6600 3150 7150 3150
+Wire Wire Line
+	7500 3350 7500 3450
+Wire Wire Line
+	7500 3450 7150 3450
+Connection ~ 7150 3050
+Wire Wire Line
+	7150 3050 7500 3050
+Wire Wire Line
+	7150 2750 7500 2750
+Connection ~ 7500 3450
 $EndSCHEMATC
