File: dac.kicad_pcb (KiCad board)
At the start: 2 copper layers, 20 parts, among them J1 RCJ-2121, J2 Conn_01x03_Male, SW1 SW_DIP_x01, U1 pcm5102a

Commit message: correcciones profe
Connections:
- C11 pad 1: GNDA -> +3.3VA
- C11 pad 2: +3.3VA -> GNDA

Commit message: ruteo PCB
Parts:
- moved C2 8.94 mm to (140.0, 100.0), turned to 90 degrees
- moved R1 8.78 mm to (153.0, 82.0), turned to 270 degrees
- moved C5 7.86 mm to (147.0, 88.0)
- moved C12 6.44 mm to (169.0, 95.0)
- moved C13 6.29 mm to (169.0, 92.0)
- moved SW1 6.19 mm to (149.0, 82.0)
- moved J1 5.45 mm to (179.0, 96.0)
- moved C6 3.79 mm to (160.0, 85.0)
- moved C3 2.24 mm to (145.8, 102.1)
- moved C4 2.00 mm to (151.0, 102.1)
- moved C10 1.99 mm to (160.0, 106.0)
- moved C1 1.79 mm to (140.0, 105.0), turned to 90 degrees
- moved C8 1.63 mm to (169.0, 86.0)
- moved C7 1.60 mm to (160.0, 100.0)
- moved R3 1.53 mm to (164.0, 95.0)
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Routing:
- net GNDA: track 0.00 -> 78.0 mm
- net +3.3VA: track 0.00 -> 61.2 mm
- net Earth: track 0.00 -> 46.1 mm
- net Net-(C9-Pad1): track 0.00 -> 21.4 mm
- net Net-(C13-Pad1): track 0.00 -> 19.8 mm
- net Net-(C1-Pad1): track 0.00 -> 19.2 mm
- net Net-(C12-Pad1): track 0.00 -> 13.5 mm
- net Net-(C7-Pad2): track 0.00 -> 12.4 mm
- net Net-(C7-Pad1): track 0.00 -> 12.0 mm
- net Net-(C5-Pad1): track 0.00 -> 11.2 mm
- net Net-(J2-Pad3): track 0.00 -> 10.4 mm
- net Net-(J2-Pad1): track 0.00 -> 10.2 mm
- net Net-(R2-Pad2): track 0.00 -> 9.66 mm
- net Net-(J2-Pad2): track 0.00 -> 9.59 mm
- net Net-(R3-Pad2): track 0.00 -> 9.26 mm
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Other:
- board outline added: 52 x 31 mm
- board text added: "11ra Cohorte - KICAD"
- board text added: "2021"

Commit message: se avanza en el pcb
Parts:
- added FID1: Fiducial, Fiducial:Fiducial_0.5mm_Mask1.5mm, F.Cu at (151.0, 97.5)
- C1, C11, C2, C8: footprint Capacitor_THT:C_Radial_D4.0mm_H5.0mm_P1.50mm -> Capacitor_THT:CP_Radial_D4.0mm_P1.50mm
Other:
- rule pad_to_mask_clearance: 0 -> 0.07
- board text added: "Decodificador Stereo Audio Digital"
- board text added: "IND. ARG. 2021"
- board text removed: "11ra Cohorte - KICAD"
- board text removed: "2021"

Commit message: se agregan comentarios de la clase 7
Parts:
- moved C9 2.11 mm to (167.0, 101.5), turned to 0 degrees
- moved C1 2.00 mm to (140.0, 103.0), turned to 270 degrees
- moved C11 1.41 mm to (167.5, 107.0), turned to 0 degrees
Routing:
- net +3.3VA: track 61.2 -> 76.6 mm
- net Earth: track 46.1 -> 60.9 mm
- net Net-(C1-Pad1): track 19.2 -> 15.3 mm
- net GNDA: track 78.0 -> 74.5 mm
- net Net-(C9-Pad1): track 21.4 -> 19.8 mm
- added copper zone on B.Cu, net GNDA
Other:
- board text added: "Grilla: 1mm, 0,5mm Margen: 0,2mm Via: 1,6mm / 0,8mm Pista: 0,2mm, 0,8mm Distancias al borde: 1mm Terminacion: HASL"

Commit message: pcb terminado
Parts:
- added J3: Conn_01x02_Male, Connector_PinHeader_2.54mm:PinHeader_1x02_P2.54mm_Vertical, F.Cu at (138.0, 83.5)
- moved J1 6.08 mm to (173.0, 95.0)
- moved C13 5.10 mm to (164.0, 91.0)
- moved C8 5.02 mm to (164.0, 85.5)
- moved C12 5.00 mm to (164.0, 95.0)
- moved C11 4.00 mm to (163.5, 107.0)
- moved C6 4.00 mm to (156.0, 85.0)
- moved C9 4.00 mm to (163.0, 101.5)
- moved R2 4.00 mm to (160.0, 91.0)
- moved R3 4.00 mm to (160.0, 95.0)
- moved J2 3.00 mm to (138.0, 91.0)
- moved C5 2.69 mm to (144.5, 89.0)
- moved C10 2.06 mm to (158.0, 105.5)
- moved C7 2.06 mm to (158.0, 100.5)
- moved SW1 2.06 mm to (148.5, 84.0)
- moved C1 2.00 mm to (142.0, 103.0)
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Connections:
- net Net-(R2-Pad2) renamed /OUTR
- net Net-(R3-Pad2) renamed /OUTL
- C1 pad 2: Earth -> GND
- C2 pad 2: Earth -> GND
- C3 pad 2: Earth -> GND
- C4 pad 1: Earth -> GND
- C5 pad 1: Net-(C5-Pad1) -> /FLT
- C5 pad 2: Earth -> GNDA
- R1 pad 1: Net-(R1-Pad1) -> +3.3VA
- R1 pad 2: Net-(C5-Pad1) -> /FLT
- SW1 pad 1: Net-(R1-Pad1) -> /FLT
- SW1 pad 2: Earth -> GNDA
- U1 pad 10: Earth -> GND
- U1 pad 11: Net-(C5-Pad1) -> /FLT
- U1 pad 12: Earth -> GND
- U1 pad 16: Earth -> GND
- U1 pad 17: Earth -> GND
- U1 pad 19: Earth -> GND
Routing:
- net Earth: track 60.9 -> 0.00 mm
- net GND: track 0.00 -> 49.4 mm, vias 0 -> 8
- net +3.3VA: track 76.6 -> 33.0 mm, vias 0 -> 8
- net GNDA: track 74.5 -> 49.6 mm, vias 0 -> 11
- net /FLT: track 0.00 -> 17.8 mm
- net Net-(C5-Pad1): track 11.2 -> 0.00 mm
- net Net-(C13-Pad1): track 19.8 -> 13.4 mm
- net Net-(R1-Pad1): track 4.00 -> 0.00 mm
- net /OUTR: track 9.66 -> 5.69 mm
- net /OUTL: track 9.26 -> 5.38 mm
- net Net-(C9-Pad1): track 19.8 -> 16.6 mm
- net Net-(J2-Pad2): track 9.59 -> 6.59 mm
- net Net-(J2-Pad3): track 10.4 -> 7.43 mm
- net Net-(J2-Pad1): track 10.2 -> 7.22 mm
- net Net-(C12-Pad1): track 13.5 -> 11.1 mm
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- added copper zone on F.Cu, net +3.3VA
Other:
- board size 52 x 31 mm -> 42 x 30 mm
- board text added: "Fabricante: Mayer Grilla: 1mm, 0,5mm Margen: 0,2mm Via: 1,6mm / 0,8mm, 0,8mm/0,40mm Pista: 0,2mm, 0,8mm Distancias al borde: 1mm Terminación superficial: HASL"
- board text removed: "Grilla: 1mm, 0,5mm Margen: 0,2mm Via: 1,6mm / 0,8mm Pista: 0,2mm, 0,8mm Distancias al borde: 1mm Terminacion: HASL"

Commit message: correcciones pcb
Parts:
- added H1: MountingHole, MountingHole:MountingHole_2.5mm, F.Cu at (138.5, 107.5)
- moved FID1 0.71 mm to (151.5, 98.0)
Routing:
- net +3.3VA: track 33.0 -> 35.9 mm
Other:
- board text added: "BCK"
- board text added: "DIN"
- board text added: "GND"
- board text added: "SCK"
- board text added: "VCC"
Changed lines of the file:
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@@
   (general
     (thickness 1.6)
-    (drawings 15)
-    (tracks 162)
+    (drawings 20)
+    (tracks 164)
     (zones 0)
-    (modules 22)
+    (modules 23)
     (nets 16)
   )
@@
   (layers
     (0 F.Cu mixed)
-    (31 B.Cu power)
+    (31 B.Cu mixed)
     (32 B.Adhes user hide)
     (33 F.Adhes user hide)
     (34 B.Paste user hide)
-    (35 F.Paste user)
+    (35 F.Paste user hide)
     (36 B.SilkS user hide)
     (37 F.SilkS user)
-    (38 B.Mask user)
+    (38 B.Mask user hide)
     (39 F.Mask user hide)
     (40 Dwgs.User user)
@@
     (add_net "Net-(J2-Pad3)")
   )
+  (module MountingHole:MountingHole_2.5mm (layer F.Cu)
+    (at 138.5 107.5)
+    (descr "Mounting Hole 2.5mm, no annular")
+    (tags "mounting hole 2.5mm no annular")
+    (attr virtual)
+    (fp_text reference H1 (at 0 -3.5) (layer F.SilkS) hide
+      (effects (font (size 1 1) (thickness 0.15)))
+    )
+    (fp_text value MountingHole (at 0 3.5) (layer F.Fab)
+      (effects (font (size 1 1) (thickness 0.15)))
+    )
+    (fp_text user %R (at 0.3 0) (layer F.Fab)
+      (effects (font (size 1 1) (thickness 0.15)))
+    )
+    (fp_circle (center 0 0) (end 2.5 0) (layer Cmts.User) (width 0.15))
+    (fp_circle (center 0 0) (end 2.75 0) (layer F.CrtYd) (width 0.05))
+    (pad 1 np_thru_hole circle (at 0 0) (size 2.5 2.5) (drill 2.5) (layers *.Cu *.Mask))
+  )
   (module Capacitor_THT:C_Disc_D3.8mm_W2.6mm_P2.50mm (layer F.Cu)
     (at 144.5 89 180)
@@
   )
   (module Fiducial:Fiducial_0.5mm_Mask1.5mm (layer F.Cu)
-    (at 151 97.5)
+    (at 151.5 98)
     (descr "Circular Fiducial, 0.5mm bare copper, 1.5mm soldermask opening")
     (tags fiducial)
@@
     )
   )
+  (gr_text SCK (at 136.4 96 90) (layer F.SilkS)
+    (effects (font (size 0.5 0.5) (thickness 0.125)))
+  )
+  (gr_text DIN (at 136.4 93.6 90) (layer F.SilkS)
+    (effects (font (size 0.5 0.5) (thickness 0.125)))
+  )
+  (gr_text BCK (at 136.4 91 90) (layer F.SilkS)
+    (effects (font (size 0.5 0.5) (thickness 0.125)))
+  )
+  (gr_text GND (at 136.4 86.2 90) (layer F.SilkS)
+    (effects (font (size 0.5 0.5) (thickness 0.125)))
+  )
+  (gr_text VCC (at 136.4 83.4 90) (layer F.SilkS)
+    (effects (font (size 0.5 0.5) (thickness 0.125)))
+  )
   (gr_line (start 178 80) (end 178 110) (layer Edge.Cuts) (width 0.1))
   (gr_line (start 136 80) (end 178 80) (layer Edge.Cuts) (width 0.1))
@@
   (segment (start 153.5 103.48) (end 158.02 108) (width 0.8) (layer F.Cu) (net 2))
   (segment (start 153.5 102.14) (end 153.5 103.48) (width 0.8) (layer F.Cu) (net 2))
-  (via (at 145.5 98) (size 0.8) (drill 0.4) (layers F.Cu B.Cu) (net 2))
-  (segment (start 144.4575 96.23) (end 144.4575 96.9575) (width 0.2) (layer F.Cu) (net 2))
-  (segment (start 144.4575 96.9575) (end 145.5 98) (width 0.2) (layer F.Cu) (net 2))
   (segment (start 150.1825 96.23) (end 149.5 96.9125) (width 0.2) (layer F.Cu) (net 2))
   (via (at 149.5 98) (size 0.8) (drill 0.4) (layers F.Cu B.Cu) (net 2))
@@
   (segment (start 153 83) (end 156 83) (width 0.8) (layer F.Cu) (net 2))
   (segment (start 161 85.5) (end 164 85.5) (width 0.8) (layer F.Cu) (net 2))
+  (via (at 144.5 98) (size 0.8) (drill 0.4) (layers F.Cu B.Cu) (net 2))
+  (segment (start 144.4575 96.23) (end 144.4575 97.9575) (width 0.2) (layer F.Cu) (net 2))
+  (segment (start 144.4575 97.9575) (end 144.5 98) (width 0.2) (layer F.Cu) (net 2))
+  (segment (start 142.5 100) (end 142 100) (width 0.2) (layer B.Cu) (net 2))
+  (segment (start 144.5 98) (end 142.5 100) (width 0.2) (layer B.Cu) (net 2))
   (segment (start 149 91.815346) (end 149 90.5) (width 0.2) (layer F.Cu) (net 3))
   (segment (start 150.1825 92.23) (end 149.414654 92.23) (width 0.2) (layer F.Cu) (net 3))
